Commit message: Controlling wheels of turtlebot3

File: turtlebot3_description/ros2_control/turtlebot3.ros2_control.xacro (robot description, xacro)
@@ -1,5 +1,5 @@
 <?xml version="1.0"?>
 <robot xmlns:xacro="http://www.ros.org/wiki/xacro">
-  <xacro:macro name="diffbot_system" params="name prefix use_fake_hardware:=^|false fake_sensor_commands:=^|false">
+  <xacro:macro name="turtlebot3_ros2_control" params="name prefix use_fake_hardware:=^|false fake_sensor_commands:=^|false">
     <ros2_control name="${name}" type="system">
       <hardware>

File: turtlebot3_description/urdf/common_properties.xacro (robot description, xacro)
@@ -1,8 +1,7 @@
 <?xml version="1.0" ?>
-<robot name="xacro_properties"
-  xmlns:xacro="http://ros.org/wiki/xacro">
+<robot name="xacro_properties" xmlns:xacro="http://ros.org/wiki/xacro">
   <!-- Init colour -->
   <material name="black">
-    <color rgba="0.0 0.0 0.0 1.0"/>
+      <color rgba="0.0 0.0 0.0 1.0"/>
   </material>
   <material name="dark">

Commit message: Adding IMU sensor

File: turtlebot3_description/ros2_control/turtlebot3.ros2_control.xacro (robot description, xacro)
@@ -31,4 +31,16 @@
         <state_interface name="velocity"/>
       </joint>
+      <sensor name="imu_sensor">
+        <state_interface name="orientation.x"/>
+        <state_interface name="orientation.y"/>
+        <state_interface name="orientation.z"/>
+        <state_interface name="orientation.w"/>
+        <state_interface name="angular_velocity.x"/>
+        <state_interface name="angular_velocity.y"/>
+        <state_interface name="angular_velocity.z"/>
+        <state_interface name="linear_acceleration.x"/>
+        <state_interface name="linear_acceleration.y"/>
+        <state_interface name="linear_acceleration.z"/>
+      </sensor>
     </ros2_control>
   </xacro:macro>

File: turtlebot3_description/urdf/turtlebot3_description.urdf.xacro (robot description, xacro)
@@ -124,8 +124,8 @@
     <joint name="imu_joint" type="fixed">
       <parent link="base_link"/>
-      <child link="imu_link"/>
+      <child link="imu_sensor"/>
       <origin xyz="0.0 0 0.068" rpy="0 0 0"/>
     </joint>
-    <link name="imu_link"/>
+    <link name="imu_sensor"/>
     <joint name="scan_joint" type="fixed">
       <parent link="base_link"/>

Commit message: Adding Gazebo support

File: turtlebot3_description/ros2_control/turtlebot3.ros2_control.xacro (robot description, xacro)
@@ -2,7 +2,7 @@
 <robot xmlns:xacro="http://www.ros.org/wiki/xacro">
   <xacro:macro name="turtlebot3_ros2_control" params="name prefix use_fake_hardware:=^|false fake_sensor_commands:=^|false">
-    <ros2_control name="${name}" type="system">
+    <ros2_control name="GazeboSystem" type="system">
       <hardware>
-        <xacro:if value="${use_fake_hardware}">
+        <!-- <xacro:if value="${use_fake_hardware}">
           <plugin>fake_components/GenericSystem</plugin>
           <param name="fake_sensor_commands">${fake_sensor_commands}</param>
@@ -13,7 +13,8 @@
           <param name="example_param_hw_start_duration_sec">2.0</param>
           <param name="example_param_hw_stop_duration_sec">3.0</param>
-        </xacro:unless>
+        </xacro:unless> -->
+        <plugin>gazebo_ros2_control/GazeboSystem</plugin>
       </hardware>
-      <joint name="${prefix}left_wheel_joint">
+      <joint name="wheel_left_joint">
         <command_interface name="velocity">
           <param name="min">-1</param>
@@ -23,5 +24,5 @@
         <state_interface name="velocity"/>
       </joint>
-      <joint name="${prefix}right_wheel_joint">
+      <joint name="wheel_right_joint">
         <command_interface name="velocity">
           <param name="min">-1</param>

File: turtlebot3_description/urdf/turtlebot3.gazebo.xacro (robot description, xacro)
@@ -4,4 +4,12 @@
   <xacro:arg name="camera_visual" default="false"/>
   <xacro:arg name="imu_visual"    default="false"/>
+  <gazebo>
+    <!-- Joint state publisher -->
+    <plugin filename="libgazebo_ros2_control.so" name="gazebo_ros2_control">
+      <robotParam>robot_description</robotParam>
+      <robot_sim_type>gazebo_ros2_control/GazeboSystem</robot_sim_type>
+      <parameters>$(find turtlebot3_bringup)/config/turtlebot3_controllers.yaml</parameters>
+    </plugin>
+  </gazebo>
   <gazebo reference="base_link">
     <material>Gazebo/DarkGrey</material>
@@ -45,6 +53,6 @@
     <material>Gazebo/FlatBlack</material>
   </gazebo>
-  <gazebo reference="imu_link">
-    <sensor type="imu" name="imu">
+  <gazebo reference="imu_sensor">
+    <sensor type="imu" name="imu_sensor">
       <always_on>true</always_on>
       <visualize>$(arg imu_visual)</visualize>
@@ -53,5 +61,5 @@
   </gazebo>
   <gazebo>
-    <plugin name="turtlebot3_waffle_controller" filename="libgazebo_ros_diff_drive.so">
+    <plugin name="turtlebot3_base_controller" filename="libgazebo_ros_diff_drive.so">
       <commandTopic>cmd_vel</commandTopic>
       <odometryTopic>odom</odometryTopic>
@@ -65,11 +73,16 @@
       <legacyMode>false</legacyMode>
       <updateRate>30</updateRate>
-      <leftJoint>wheel_left_joint</leftJoint>
-      <rightJoint>wheel_right_joint</rightJoint>
-      <wheelSeparation>0.287</wheelSeparation>
-      <wheelDiameter>0.066</wheelDiameter>
-      <wheelAcceleration>1</wheelAcceleration>
-      <wheelTorque>10</wheelTorque>
+      <left_joint>wheel_left_joint</left_joint>
+      <right_joint>wheel_right_joint</right_joint>
+      <wheel_separation>0.287</wheel_separation>
+      <wheel_diameter>0.066</wheel_diameter>
+      <max_wheel_acceleration>1</max_wheel_acceleration>
+      <max_wheel_torque>10</max_wheel_torque>
       <rosDebugLevel>na</rosDebugLevel>
+            <!-- output -->
+      <publish_odom>true</publish_odom>
+      <publish_odom_tf>true</publish_odom_tf>
+      <odometry_frame>odom</odometry_frame>
+      <robot_base_frame>chassis</robot_base_frame>
     </plugin>
   </gazebo>
@@ -77,6 +90,6 @@
     <plugin name="imu_plugin" filename="libgazebo_ros_imu.so">
       <alwaysOn>true</alwaysOn>
-      <bodyName>imu_link</bodyName>
-      <frameName>imu_link</frameName>
+      <bodyName>imu_sensor</bodyName>
+      <frameName>imu_sensor</frameName>
       <topicName>imu</topicName>
       <serviceName>imu_service</serviceName>

Commit message: Fix odom publishing problem

File: turtlebot3_description/ros2_control/turtlebot3.ros2_control.xacro (robot description, xacro)
@@ -1,19 +1,25 @@
 <?xml version="1.0"?>
 <robot xmlns:xacro="http://www.ros.org/wiki/xacro">
-  <xacro:macro name="turtlebot3_ros2_control" params="name prefix use_fake_hardware:=^|false fake_sensor_commands:=^|false">
+  <xacro:macro name="turtlebot3_ros2_control" params="name prefix use_sim_time:=^|false use_fake_hardware:=^|false fake_sensor_commands:=^|false">
     <ros2_control name="GazeboSystem" type="system">
-      <hardware>
-        <!-- <xacro:if value="${use_fake_hardware}">
-          <plugin>fake_components/GenericSystem</plugin>
-          <param name="fake_sensor_commands">${fake_sensor_commands}</param>
-          <param name="state_following_offset">0.0</param>
-        </xacro:if>
-        <xacro:unless value="${use_fake_hardware}">
-          <plugin>turtlebot3_hardware/TurtleBot3Hardware</plugin>
-          <param name="example_param_hw_start_duration_sec">2.0</param>
-          <param name="example_param_hw_stop_duration_sec">3.0</param>
-        </xacro:unless> -->
-        <plugin>gazebo_ros2_control/GazeboSystem</plugin>
-      </hardware>
+      <xacro:if value="$(arg use_sim_time)">
+        <hardware>
+          <plugin>gazebo_ros2_control/GazeboSystem</plugin>
+        </hardware>
+      </xacro:if>
+      <xacro:unless value="$(arg use_sim_time)">
+        <hardware>
+          <xacro:if value="${use_fake_hardware}">
+            <plugin>fake_components/GenericSystem</plugin>
+            <param name="fake_sensor_commands">${fake_sensor_commands}</param>
+            <param name="state_following_offset">0.0</param>
+          </xacro:if>
+          <xacro:unless value="${use_fake_hardware}">
+            <plugin>turtlebot3_hardware/TurtleBot3Hardware</plugin>
+            <param name="example_param_hw_start_duration_sec">2.0</param>
+            <param name="example_param_hw_stop_duration_sec">3.0</param>
+          </xacro:unless>
+        </hardware>
+      </xacro:unless>
       <joint name="wheel_left_joint">
         <command_interface name="velocity">

File: turtlebot3_description/urdf/turtlebot3.gazebo.xacro (robot description, xacro)
@@ -59,30 +59,4 @@
     </sensor>
     <material>Gazebo/Grey</material>
-  </gazebo>
-  <gazebo>
-    <plugin name="turtlebot3_base_controller" filename="libgazebo_ros_diff_drive.so">
-      <commandTopic>cmd_vel</commandTopic>
-      <odometryTopic>odom</odometryTopic>
-      <odometryFrame>odom</odometryFrame>
-      <odometrySource>world</odometrySource>
-      <publishOdomTF>true</publishOdomTF>
-      <robotBaseFrame>base_footprint</robotBaseFrame>
-      <publishWheelTF>false</publishWheelTF>
-      <publishTf>true</publishTf>
-      <publishWheelJointState>true</publishWheelJointState>
-      <legacyMode>false</legacyMode>
-      <updateRate>30</updateRate>
-      <left_joint>wheel_left_joint</left_joint>
-      <right_joint>wheel_right_joint</right_joint>
-      <wheel_separation>0.287</wheel_separation>
-      <wheel_diameter>0.066</wheel_diameter>
-      <max_wheel_acceleration>1</max_wheel_acceleration>
-      <max_wheel_torque>10</max_wheel_torque>
-      <rosDebugLevel>na</rosDebugLevel>
-            <!-- output -->
-      <publish_odom>true</publish_odom>
-      <publish_odom_tf>true</publish_odom_tf>
-      <odometry_frame>odom</odometry_frame>
-    </plugin>
   </gazebo>
   <gazebo>

File: turtlebot3_description/urdf/turtlebot3.urdf.xacro (robot description, xacro)
@@ -1,6 +1,8 @@
 <?xml version="1.0"?>
 <!-- Basic differential drive mobile base -->
-<robot xmlns:xacro="http://www.ros.org/wiki/xacro" name="diffdrive_robot">
+<robot xmlns:xacro="http://www.ros.org/wiki/xacro" name="turtlebot3_robot">
   <xacro:arg name="prefix" default="" />
+  <xacro:arg name="use_sim_time" default="false" />
+  <xacro:arg name="use_fake_hardware" default="false" />
   <xacro:include filename="$(find turtlebot3_description)/urdf/turtlebot3_description.urdf.xacro" />
   <xacro:include filename="$(find turtlebot3_description)/urdf/turtlebot3.gazebo.xacro"/>
@@ -11,4 +13,7 @@
   <xacro:turtlebot3 prefix="$(arg prefix)" />
   <xacro:turtlebot3_ros2_control
-    name="turtlebot3" prefix="$(arg prefix)" />
+    name="turtlebot3" prefix="$(arg prefix)"
+    use_fake_hardware="$(arg use_fake_hardware)"
+    use_sim_time="$(arg use_sim_time)"
+  />
 </robot>
